Commit message: 20190726 ナビゲーション実装

File: robot_pkg/urdf/wheel_robot_base.urdf.xacro (robot description, xacro)
@@ -12,4 +12,5 @@
   <property name="base_z_size" value="0.25" />
   <property name="base_mass" value="35" /> <!-- in kg-->
+  <property name="hokuyo_size" value="0.1" />
   <!--Inertial macros for the box and cylinder. Units are kg*m^2-->
   <macro name="box_inertia" params="m x y z">
@@ -70,4 +71,50 @@
     <turnGravityOff>false</turnGravityOff>
   </gazebo>
+  <link name="hokuyo_link">
+    <visual>
+      <origin xyz="0 0 0" rpy="0 0 0" />
+      <geometry>
+        <box size="${hokuyo_size} ${hokuyo_size} ${hokuyo_size}"/>
+	<!--box size="0.05 0.05 0.05"/-->
+      </geometry>
+      <material name="Blue" />
+    </visual>
+  </link>
+  <joint name="hokuyo_joint" type="fixed">
+    <origin xyz="${hokuyo_size/2} 0 ${0.2+hokuyo_size/4}" rpy="0 0 0" />
+    <!--origin xyz="${0.05/2} 0 ${0.2+0.05/4}" rpy="0 0 0" /-->
+    <parent link="base_link"/>
+    <child link="hokuyo_link" />
+  </joint>
+  <gazebo reference="hokuyo_link">
+    <material>Gazebo/Blue</material>
+    <turnGravityOff>false</turnGravityOff>
+    <sensor type="ray" name="head_hokuyo_sensor">
+      <pose>${hokuyo_size/2} 0 0 0 0 0</pose>
+      <!--pose>${0.05/2} 0 0 0 0 0</pose-->
+      <visualize>false</visualize>
+      <update_rate>40</update_rate>
+      <ray>
+        <scan>
+          <horizontal>
+            <samples>720</samples>
+            <resolution>1</resolution>
+            <min_angle>-1.570796</min_angle>
+            <max_angle>1.570796</max_angle>
+          </horizontal>
+        </scan>
+        <range>
+          <min>0.10</min>
+          <max>10.0</max>
+          <resolution>0.001</resolution>
+        </range>
+      </ray>
+      <plugin name="gazebo_ros_head_hokuyo_controller" filename="libgazebo_ros_laser.so">
+        <topicName>/scan</topicName>
+        <frameName>hokuyo_link</frameName>
+	<legacyModeNS>true</legacyModeNS>
+      </plugin>
+    </sensor>
+  </gazebo>
   <!-- WHEELs -->
   <wheel fb="front" lr="right" parent="base_link" translateX="1" translateY="-1" flipY="-1"/>
@@ -91,4 +138,5 @@
       <odometryTopic>odom</odometryTopic>
       <robotBaseFrame>base_footprint</robotBaseFrame>
+      <legacyModeNS>true</legacyModeNS>
     </plugin>
     <plugin name="gazebo_ros_control" filename="libgazebo_ros_control.so" />
